File: eagle/nibblet.brd (EAGLE design)
At the start: 31.3 x 31.2 mm, 37 parts, among them IC1 MEGA8-AI

Commit message: pin checking, LED array
Parts:
- added IC2: AT90S2313S, atmel:SO20L
- added LED15, LED16, LED17, LED18, LED19, LED20, LED21, LED22, LED23, LED24, LED25, LED26, LED27, LED28: (no value), led:CHIP-LED0805
Connections:
- new net N$37: LED15.C, LED19.C, LED23.C, LED27.C
- new net N$38: LED27.A, LED28.A
- new net N$39: LED23.A, LED24.A, LED25.A, LED26.A
- new net N$40: LED19.A, LED20.A, LED21.A, LED22.A
- new net N$41: LED15.A, LED16.A, LED17.A, LED18.A
- new net N$42: LED16.C, LED20.C, LED24.C, LED28.C
- new net N$43: LED17.C, LED21.C, LED25.C
- new net N$44: LED18.C, LED22.C, LED26.C
- net GND: now also IC2.10
- net VCC: now also IC2.20
Changed lines of the file:
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@@
 <element name="PAD2" library="wirepad" package="SMD1,27-2,54" value="WIREPADSMD1,27-254" x="16.4" y="7.8" rot="MR150"/>
 <element name="PAD3" library="wirepad" package="SMD1,27-2,54" value="WIREPADSMD1,27-254" x="16.4" y="9.8" rot="MR30"/>
+<element name="IC2" library="atmel" package="SO20L" value="AT90S2313S" x="7.6" y="-5.7">
+<attribute name="OC_NEWARK" value="unknown" x="7.6" y="-5.7" size="1.778" layer="27" display="off"/>
+<attribute name="MPN" value="" x="7.6" y="-5.7" size="1.778" layer="27" display="off"/>
+<attribute name="MF" value="" x="7.6" y="-5.7" size="1.778" layer="27" display="off"/>
+<attribute name="OC_FARNELL" value="unknown" x="7.6" y="-5.7" size="1.778" layer="27" display="off"/>
+</element>
+<element name="LED15" library="led" package="CHIP-LED0805" value="" x="2.2" y="-16.3"/>
+<element name="LED16" library="led" package="CHIP-LED0805" value="" x="6.2" y="-16.3"/>
+<element name="LED17" library="led" package="CHIP-LED0805" value="" x="10.2" y="-16.3"/>
+<element name="LED18" library="led" package="CHIP-LED0805" value="" x="14.2" y="-16.3"/>
+<element name="LED19" library="led" package="CHIP-LED0805" value="" x="2.2" y="-22.9"/>
+<element name="LED20" library="led" package="CHIP-LED0805" value="" x="6.2" y="-22.9"/>
+<element name="LED21" library="led" package="CHIP-LED0805" value="" x="10.2" y="-22.9"/>
+<element name="LED22" library="led" package="CHIP-LED0805" value="" x="14.2" y="-22.9"/>
+<element name="LED23" library="led" package="CHIP-LED0805" value="" x="2.2" y="-29.5"/>
+<element name="LED24" library="led" package="CHIP-LED0805" value="" x="6.2" y="-29.5"/>
+<element name="LED25" library="led" package="CHIP-LED0805" value="" x="10.2" y="-29.5"/>
+<element name="LED26" library="led" package="CHIP-LED0805" value="" x="14.2" y="-29.5"/>
+<element name="LED27" library="led" package="CHIP-LED0805" value="" x="2.2" y="-36.1"/>
+<element name="LED28" library="led" package="CHIP-LED0805" value="" x="6.2" y="-36.1"/>
 </elements>
 <signals>
@@
 <via x="20.9" y="24.4" extent="1-16" drill="0.3"/>
 <via x="21.7" y="22" extent="1-16" drill="0.3"/>
+<contactref element="IC2" pad="20"/>
+<wire x1="2.52" y1="-1.3058" x2="28.7" y2="11.8" width="0" layer="19" extent="1-16"/>
 </signal>
 <signal name="GND">
@@
 <wire x1="16.4" y1="8" x2="16.4" y2="7.8" width="0.4064" layer="16"/>
 <wire x1="14.3" y1="8.7" x2="15.7" y2="8.7" width="0.4064" layer="16"/>
+<contactref element="IC2" pad="10"/>
+<wire x1="13.95" y1="-10.8308" x2="13.6" y2="5.7" width="0" layer="19" extent="1-1"/>
 </signal>
 <signal name="N$19">
@@
 <via x="7.2" y="14.3" extent="1-16" drill="0.3"/>
 </signal>
+<signal name="N$37">
+<contactref element="LED27" pad="C"/>
+<contactref element="LED23" pad="C"/>
+<contactref element="LED19" pad="C"/>
+<contactref element="LED15" pad="C"/>
+<wire x1="2.2" y1="-28.45" x2="2.2" y2="-35.05" width="0" layer="19" extent="1-1"/>
+<wire x1="2.2" y1="-21.85" x2="2.2" y2="-28.45" width="0" layer="19" extent="1-1"/>
+<wire x1="2.2" y1="-15.25" x2="2.2" y2="-21.85" width="0" layer="19" extent="1-1"/>
+</signal>
+<signal name="N$38">
+<contactref element="LED27" pad="A"/>
+<contactref element="LED28" pad="A"/>
+<wire x1="6.2" y1="-37.15" x2="2.2" y2="-37.15" width="0" layer="19" extent="1-1"/>
+</signal>
+<signal name="N$39">
+<contactref element="LED23" pad="A"/>
+<contactref element="LED24" pad="A"/>
+<contactref element="LED25" pad="A"/>
+<contactref element="LED26" pad="A"/>
+<wire x1="6.2" y1="-30.55" x2="2.2" y2="-30.55" width="0" layer="19" extent="1-1"/>
+<wire x1="10.2" y1="-30.55" x2="6.2" y2="-30.55" width="0" layer="19" extent="1-1"/>
+<wire x1="14.2" y1="-30.55" x2="10.2" y2="-30.55" width="0" layer="19" extent="1-1"/>
+</signal>
+<signal name="N$40">
+<contactref element="LED19" pad="A"/>
+<contactref element="LED20" pad="A"/>
+<contactref element="LED21" pad="A"/>
+<contactref element="LED22" pad="A"/>
+<wire x1="6.2" y1="-23.95" x2="2.2" y2="-23.95" width="0" layer="19" extent="1-1"/>
+<wire x1="10.2" y1="-23.95" x2="6.2" y2="-23.95" width="0" layer="19" extent="1-1"/>
+<wire x1="14.2" y1="-23.95" x2="10.2" y2="-23.95" width="0" layer="19" extent="1-1"/>
+</signal>
+<signal name="N$41">
+<contactref element="LED15" pad="A"/>
+<contactref element="LED16" pad="A"/>
+<contactref element="LED17" pad="A"/>
+<contactref element="LED18" pad="A"/>
+<wire x1="6.2" y1="-17.35" x2="2.2" y2="-17.35" width="0" layer="19" extent="1-1"/>
+<wire x1="10.2" y1="-17.35" x2="6.2" y2="-17.35" width="0" layer="19" extent="1-1"/>
+<wire x1="14.2" y1="-17.35" x2="10.2" y2="-17.35" width="0" layer="19" extent="1-1"/>
+</signal>
+<signal name="N$42">
+<contactref element="LED28" pad="C"/>
+<contactref element="LED24" pad="C"/>
+<contactref element="LED20" pad="C"/>
+<contactref element="LED16" pad="C"/>
+<wire x1="6.2" y1="-28.45" x2="6.2" y2="-35.05" width="0" layer="19" extent="1-1"/>
+<wire x1="6.2" y1="-21.85" x2="6.2" y2="-28.45" width="0" layer="19" extent="1-1"/>
+<wire x1="6.2" y1="-15.25" x2="6.2" y2="-21.85" width="0" layer="19" extent="1-1"/>
+</signal>
+<signal name="N$43">
+<contactref element="LED25" pad="C"/>
+<contactref element="LED21" pad="C"/>
+<contactref element="LED17" pad="C"/>
+<wire x1="10.2" y1="-21.85" x2="10.2" y2="-28.45" width="0" layer="19" extent="1-1"/>
+<wire x1="10.2" y1="-15.25" x2="10.2" y2="-21.85" width="0" layer="19" extent="1-1"/>
+</signal>
+<signal name="N$44">
+<contactref element="LED26" pad="C"/>
+<contactref element="LED22" pad="C"/>
+<contactref element="LED18" pad="C"/>
+<wire x1="14.2" y1="-21.85" x2="14.2" y2="-28.45" width="0" layer="19" extent="1-1"/>
+<wire x1="14.2" y1="-15.25" x2="14.2" y2="-21.85" width="0" layer="19" extent="1-1"/>
+</signal>
 </signals>
